File: hardware/led-pedestal.kicad_sch (KiCad schematic)
At the start: 29 parts, among them J1 USB_B_Micro, J2 ISP, Q1 AO3401A, SW1 SKRPACE010, U1 LTC4054ES5-4.2, U2 FS8205A, U3 FS312F-G, U4 XC6206PxxxMR, U5 PIC10F222-IOT

Commit message: Add revision 2 of the hardware
Changes include:
- moved button to the center for better fit of the case
- added silkscreen marks for + and minus of the LED
- connect jumper to battery measurement variant
- lower charging current (from 100 to 30 mA)
Parts:
- removed C3: 100n|10k, Capacitor_SMD:C_0805_2012Metric_Pad1.18x1.45mm_HandSolder, symbol Device:C
- removed JP1: Variant select jumper, Jumper:SolderJumper-3_P1.3mm_Open_RoundedPad1.0x1.5mm, symbol Jumper:Jumper_3_Open
- removed TH1: 10k|33k, Resistor_SMD:R_0805_2012Metric_Pad1.20x1.40mm_HandSolder, symbol Device:Thermistor
- added JP1: Variant select jumper, Jumper:SolderJumper-3_P1.3mm_Bridged12_RoundedPad1.0x1.5mm_NumberLabels, symbol Jumper:SolderJumper_3_Bridged12
- added R8: 33k, Resistor_SMD:R_0805_2012Metric_Pad1.20x1.40mm_HandSolder, symbol Device:R
- added R9: 10k, Resistor_SMD:R_0805_2012Metric_Pad1.20x1.40mm_HandSolder, symbol Device:R
- R1: value 10k -> 33k
- R6: value 470 -> 100
- U1: value LTC4054ES5-4.2 -> LTC4054|TP4054
Connections:
- net +BATT: now also JP1.1 (A)
- net AN1|CLK: now also R8.2, R9.2
- net GND: now also JP1.3 (B), R8.1
- new net: JP1.2 (C), R9.1
Other:
- note added: "30 mA charge current"
- note added: "Variant 1: Battery voltage measurement resistor divider network"
- note added: "Variant 2: Random seed generator based on RC time constant 10k NTC thermistor in place of R8 100nF capacitor in place of R9"
- note added: "Variant select To VBAT: Variant 1 To GND: Variant 2"
- note removed: "100 mA charge current"
- note removed: "Variant 1: Random seed generator based on RC time constant"
- note removed: "Variant 2: Battery Voltage masurement Resistor divider network instead of thermistor and capacitor 33k resistor in place of TH1 10k resistor in place of C3"
- note removed: "Variant select To GND: Variant 1 To VBAT: Variant 2"
- company: (none) -> Galion
- title: (none) -> LED Pedestal
